Commit message: working on robot model (moveit package, fixes on the urdf model)

File: robocluedo_dependencies/robocluedo_urdf_model/model/robocluedo_urdf.urdf (robot description, URDF)
Before this commit: robot robocluedo_robot, 11 links, 10 joints
Links:
- link cluedo_link: mass 0.025 -> 0.015
Joints:
- joint arm_joint_04: origin xyz=0 0 0.15 rpy=0 0 0 -> xyz=0 0 0.3 rpy=0 0 0
- joint left_grip_joint: origin xyz=-0.015 0 0.15 rpy=0 0 0 -> xyz=-0.015 0 0.0 rpy=0 0 0
- joint right_grip_joint: origin xyz=-0.015 0 0.15 rpy=0 0 0 -> xyz=-0.015 0 0.0 rpy=0 0 0

File: robocluedo_dependencies/robocluedo_urdf_model/robocluedo_arm_gripper.xacro (robot description, xacro)
@@ -3,10 +3,10 @@
     <link name="cluedo_link">
 <inertial>
-            <mass value="0.025" />
-            <origin rpy="0 0 0" xyz="0 0 0.15" />
+            <mass value="0.015" />
+            <origin rpy="0 0 0" xyz="0 0 0" />
             <inertia ixx="0.000010279" ixy="0" ixz="0" iyy="0.000010279" iyz="0" izz="0.000007225" />
         </inertial>
         <collision>
-            <origin rpy="0 0 1.57" xyz="0 0 0.15" />
+            <origin rpy="0 0 1.57" xyz="0 0 0.04" />
             <geometry>
                 <box size="0.034 0.2 0.08" />
@@ -14,5 +14,5 @@
         </collision>
         <visual>
-            <origin rpy="0 0 1.57" xyz="0 0 0.15" />
+            <origin rpy="0 0 1.57" xyz="0 0 0.04" />
             <geometry>
                 <box size="0.034 0.2 0.08" />
@@ -24,5 +24,5 @@
         <axis xyz="1 0 0" />
         <limit effort="1000.0" lower="-1.8" upper="1.8" velocity="0.5" />
-        <origin rpy="0 0 0" xyz="0 0 0.15" />
+        <origin rpy="0 0 0" xyz="0 0 0.3" />
         <parent link="arm_link_03" />
         <child link="cluedo_link" />
@@ -35,5 +35,5 @@
         </inertial>
         <collision>
-            <origin rpy="0 3.1415 -1.57" xyz="-0.032 0.048 0.0" />
+            <origin rpy="0 3.1415 -1.57" xyz="-0.032 0.048 0.04" />
             <geometry>
                 <box size="0.06 0.02 0.08" />
@@ -41,5 +41,5 @@
         </collision>
         <visual>
-            <origin rpy="0 3.1415 -1.57" xyz="-0.032 0.048 0.0" />
+            <origin rpy="0 3.1415 -1.57" xyz="-0.032 0.048 0.04" />
             <geometry>
                 <box size="0.06 0.02 0.08" />
@@ -51,5 +51,5 @@
         <axis xyz="1 0 0" />
         <limit effort="1000.0" lower="-0.04" upper="0.035" velocity="6.5" />
-        <origin rpy="0 0 0" xyz="-0.015 0 0.15" />
+        <origin rpy="0 0 0" xyz="-0.015 0 0.0" />
         <parent link="cluedo_link" />
         <child link="right_grip_link" />
@@ -62,5 +62,5 @@
         </inertial>
         <collision>
-            <origin rpy="0 3.1415 -1.57" xyz="0.06 0.048 0.0" />
+            <origin rpy="0 3.1415 -1.57" xyz="0.06 0.048 0.04" />
             <geometry>
                 <box size="0.06 0.02 0.08" />
@@ -68,5 +68,5 @@
         </collision>
         <visual>
-            <origin rpy="0 3.1415 -1.57" xyz="0.06 0.048 0.0" />
+            <origin rpy="0 3.1415 -1.57" xyz="0.06 0.048 0.04" />
             <geometry>
                 <box size="0.06 0.02 0.08" />
@@ -78,5 +78,5 @@
         <axis xyz="1 0 0" />
         <limit effort="1000.0" lower="-0.035" upper="0.04" velocity="6.5" />
-        <origin rpy="0 0 0" xyz="-0.015 0 0.15" />
+        <origin rpy="0 0 0" xyz="-0.015 0 0.0" />
         <parent link="cluedo_link" />
         <child link="left_grip_link" />
