Commit message: working on robot model (improving the stability of the robot)

File: robocluedo_dependencies/robocluedo_urdf_model/robot/model/robocluedo_urdf.urdf (robot description, URDF)
Before this commit: robot robocluedo_robot, 11 links, 10 joints
Links:
- removed link left_grip_link
- removed link right_grip_link
- added link link_a_left_wheel, mass 0.2; collision cylinder length=0.04 radius=0.1; visual cylinder length=0.04 radius=0.1
- added link link_a_right_wheel, mass 0.2; collision cylinder length=0.04 radius=0.1; visual cylinder length=0.04 radius=0.1
- link base_link: geometry collision box size=0.5 0.3 0.07; visual box size=0.5 0.3 0.07
Joints:
- removed joint left_grip_joint
- removed joint right_grip_joint
- added joint joint_a_left_wheel: type continuous, parent base_link, child link_a_left_wheel, origin xyz=-0.2 -0.15 0 rpy=0 0 0, axis 0 1 0, limit effort=10000 velocity=1000
- added joint joint_a_right_wheel: type continuous, parent base_link, child link_a_right_wheel, origin xyz=-0.2 0.15 0 rpy=0 0 0, axis 0 1 0, limit effort=10000 velocity=1000
- joint arm_base_to_base: origin xyz=0 0 0.085 rpy=0 0 0 -> xyz=-0.075 0 0.085 rpy=0 0 0
- joint joint_left_wheel: origin xyz=-0.05 -0.15 0 rpy=0 0 0 -> xyz=0.125 -0.15 0 rpy=0 0 0
- joint joint_right_wheel: origin xyz=-0.05 0.15 0 rpy=0 0 0 -> xyz=0.125 0.15 0 rpy=0 0 0

File: robocluedo_dependencies/robocluedo_urdf_model/robot/robocluedo_arm.xacro (robot description, xacro)
@@ -2,5 +2,5 @@
 <robot name="robocluedo_robot" xmlns:xacro="http://www.ros.org/wiki/xacro">
     <link name="arm_base_link">
-<inertial>
+		<inertial>
             <mass value="0.1" />
             <origin rpy="0 0 0" xyz="0 0 0" />
@@ -22,10 +22,10 @@
     </link>
     <joint name="arm_base_to_base" type="fixed">
-        <origin rpy="0 0 0" xyz="0 0 0.085" />
+        <origin rpy="0 0 0" xyz="-0.075 0 0.085" />
         <parent link="base_link" />
         <child link="arm_base_link" />
     </joint>
     <link name="arm_link_01">
-<inertial>
+		<inertial>
             <mass value="0.025" />
             <origin rpy="0 0 0" xyz="0 0 0.15" />

File: robocluedo_dependencies/robocluedo_urdf_model/robot/robocluedo_arm_gripper.xacro (robot description, xacro)
@@ -2,5 +2,5 @@
 <robot name="robocluedo_robot" xmlns:xacro="http://www.ros.org/wiki/xacro">
     <link name="cluedo_link">
-<inertial>
+		<inertial>
             <mass value="0.015" />
             <origin rpy="0 0 0" xyz="0 0 0" />
@@ -28,4 +28,5 @@
         <child link="cluedo_link" />
     </joint>
+<!--
     <link name="right_grip_link">
 <inertial>
@@ -82,3 +83,4 @@
         <child link="left_grip_link" />
     </joint>
+-->
 </robot>

File: robocluedo_dependencies/robocluedo_urdf_model/robot/robocluedo_chassis.xacro (robot description, xacro)
@@ -4,5 +4,5 @@
         <!-- pose and inertial -->
         <pose>0 0 0.1 0 0 0</pose>
-<inertial>
+		<inertial>
             <mass value="0.5" />
             <origin rpy="0 0 0" xyz="0 0 0.1" />
@@ -23,6 +23,7 @@
         </visual>
         <!-- caster front collision -->
+        <!--
         <collision name="caster_front_collision">
-            <origin rpy=" 0 0 0" xyz="0.35 0 -0.05" />
+            <origin rpy=" 0 0 0" xyz="-0.35 0 -0.05" />
             <geometry>
                 <sphere radius="0.05" />
@@ -40,12 +41,13 @@
         </collision>
         <visual name="caster_front_visual">
-            <origin rpy=" 0 0 0" xyz="0.2 0 -0.05" />
+            <origin rpy=" 0 0 0" xyz="-0.2 0 -0.05" />
             <geometry>
                 <sphere radius="0.05" />
             </geometry>
         </visual>
+        -->
     </link>
     <link name="link_right_wheel">
-<inertial>
+		<inertial>
             <mass value="0.2" />
             <origin rpy="0 1.5707 1.5707" xyz="0 0 0" />
@@ -66,5 +68,5 @@
     </link>
     <link name="link_left_wheel">
-<inertial>
+		<inertial>
             <mass value="0.2" />
             <origin rpy="0 1.5707 1.5707" xyz="0 0 0" />
@@ -85,5 +87,5 @@
     </link>
     <joint name="joint_right_wheel" type="continuous">
-        <origin rpy="0 0 0" xyz="-0.05 0.15 0" />
+        <origin rpy="0 0 0" xyz="0.125 0.15 0" />
         <child link="link_right_wheel" />
         <parent link="base_link" />
@@ -93,5 +95,5 @@
     </joint>
     <joint name="joint_left_wheel" type="continuous">
-        <origin rpy="0 0 0" xyz="-0.05 -0.15 0" />
+        <origin rpy="0 0 0" xyz="0.125 -0.15 0" />
         <child link="link_left_wheel" />
         <parent link="base_link" />
@@ -100,3 +102,57 @@
         <joint_properties damping="1.0" friction="1.0" />
     </joint>
+    <link name="link_a_right_wheel">
+		<inertial>
+            <mass value="0.2" />
+            <origin rpy="0 1.5707 1.5707" xyz="0 0 0" />
+            <inertia ixx="0.000526666666667" ixy="0" ixz="0" iyy="0.000526666666667" iyz="0" izz="0.001" />
+        </inertial>
+        <collision name="link_right_wheel_collision">
+            <origin rpy="0 1.5707 1.5707" xyz="0 0 0" />
+            <geometry>
+                <cylinder length="0.04" radius="0.1" />
+            </geometry>
+        </collision>
+        <visual name="link_right_wheel_visual">
+            <origin rpy="0 1.5707 1.5707" xyz="0 0 0" />
+            <geometry>
+                <cylinder length="0.04" radius="0.1" />
+            </geometry>
+        </visual>
+    </link>
+    <link name="link_a_left_wheel">
+		<inertial>
+            <mass value="0.2" />
+            <origin rpy="0 1.5707 1.5707" xyz="0 0 0" />
+            <inertia ixx="0.000526666666667" ixy="0" ixz="0" iyy="0.000526666666667" iyz="0" izz="0.001" />
+        </inertial>
+        <collision name="link_right_wheel_collision">
+            <origin rpy="0 1.5707 1.5707" xyz="0 0 0" />
+            <geometry>
+                <cylinder length="0.04" radius="0.1" />
+            </geometry>
+        </collision>
+        <visual name="link_left_wheel_visual">
+            <origin rpy="0 1.5707 1.5707" xyz="0 0 0" />
+            <geometry>
+                <cylinder length="0.04" radius="0.1" />
+            </geometry>
+        </visual>
+    </link>
+    <joint name="joint_a_right_wheel" type="continuous">
+        <origin rpy="0 0 0" xyz="-0.2 0.15 0" />
+        <child link="link_a_right_wheel" />
+        <parent link="base_link" />
+        <axis rpy="0 0 0" xyz="0 1 0" />
+        <limit effort="10000" velocity="1000" />
+        <joint_properties damping="1.0" friction="1.0" />
+    </joint>
+    <joint name="joint_a_left_wheel" type="continuous">
+        <origin rpy="0 0 0" xyz="-0.2 -0.15 0" />
+        <child link="link_a_left_wheel" />
+        <parent link="base_link" />
+        <axis rpy="0 0 0" xyz="0 1 0" />
+        <limit effort="10000" velocity="1000" />
+        <joint_properties damping="1.0" friction="1.0" />
+    </joint>
 </robot>

File: robocluedo_dependencies/robocluedo_urdf_model/robot/robocluedo_gazebo_materials.xacro (robot description, xacro)
@@ -52,4 +52,10 @@
         <material>Gazebo/Blue</material>
     </gazebo>
+    <gazebo reference="link_a_left_wheel">
+        <material>Gazebo/Blue</material>
+    </gazebo>
+    <gazebo reference="link_a_right_wheel">
+        <material>Gazebo/Blue</material>
+    </gazebo>
     <gazebo reference="arm_base_link">
         <material>Gazebo/Red</material>
@@ -70,4 +76,5 @@
         <material>Gazebo/Red</material>
     </gazebo>
+    <!--
     <gazebo reference="right_grip_link">
         <material>Gazebo/White</material>
@@ -76,3 +83,4 @@
         <material>Gazebo/White</material>
     </gazebo>
+    -->
 </robot>

File: robocluedo_dependencies/robocluedo_urdf_model/robot/robocluedo_sensing.xacro (robot description, xacro)
@@ -2,5 +2,5 @@
 <robot name="robocluedo_robot" xmlns:xacro="http://www.ros.org/wiki/xacro">
     <link name="laser">
-<inertial>
+		<inertial>
             <origin rpy="0 0 0" xyz="0 0 0" />
             <mass value="1" />

File: robocluedo_dependencies/robocluedo_urdf_model/robot/robocluedo_transmission.xacro (robot description, xacro)
@@ -41,4 +41,5 @@
         </actuator>
     </transmission>
+    <!--
     <transmission name="left_grip_trans">
         <type>transmission_interface/SimpleTransmission</type>
@@ -61,4 +62,5 @@
         </actuator>
     </transmission>
+    -->
     <transmission name="trans_joint_right_wheel">
         <type>transmission_interface/SimpleTransmission</type>
@@ -121,4 +123,5 @@
         </actuator>
     </transmission>
+    <!--
     <transmission name="trans_right_grip_joint">
         <type>transmission_interface/SimpleTransmission</type>
@@ -141,3 +144,4 @@
         </actuator>
     </transmission>
+    -->
 </robot>

Commit message: working on robot model and navigation (stability and behavioural improvements)

File: robocluedo_dependencies/robocluedo_urdf_model/robot/model/robocluedo_urdf.urdf (robot description, URDF)
Before this commit: robot robocluedo_robot, 11 links, 10 joints
Joints:
- joint joint_a_left_wheel: origin xyz=-0.2 -0.15 0 rpy=0 0 0 -> xyz=-0.12 -0.15 0 rpy=0 0 0
- joint joint_a_right_wheel: origin xyz=-0.2 0.15 0 rpy=0 0 0 -> xyz=-0.12 0.15 0 rpy=0 0 0

File: robocluedo_dependencies/robocluedo_urdf_model/robot/robocluedo_chassis.xacro (robot description, xacro)
@@ -141,5 +141,5 @@
     </link>
     <joint name="joint_a_right_wheel" type="continuous">
-        <origin rpy="0 0 0" xyz="-0.2 0.15 0" />
+        <origin rpy="0 0 0" xyz="-0.12 0.15 0" />
         <child link="link_a_right_wheel" />
         <parent link="base_link" />
@@ -149,5 +149,5 @@
     </joint>
     <joint name="joint_a_left_wheel" type="continuous">
-        <origin rpy="0 0 0" xyz="-0.2 -0.15 0" />
+        <origin rpy="0 0 0" xyz="-0.12 -0.15 0" />
         <child link="link_a_left_wheel" />
         <parent link="base_link" />
